File: Hardware/Qwiic_UV_Sensor_VEML6075.brd (EAGLE design)
At the start: 38.1 x 25.4 mm, 53 parts, among them J1 GATORGATOR_MINI, J2 GATORGATOR_MINI, J3 GATORGATOR_MINI, J4 GATORGATOR_MINI, J5 GATORGATOR_MINI, J6 GATORGATOR_MINI, J7 GATORGATOR_MINI, J8 GATORGATOR_MINI, Q1 2.5A/30V/105mΩ, U1 VEML6070"

Commit message: engineer run of checklist
Parts:
- removed U$16: (no value), Labels:PWR-()-03
- added U$25: (no value), buzzard_labels (13):PWR0
- moved R3 2.29 mm to (21.0, 10.2)
- moved C4 2.01 mm to (17.1, 10.2), turned to 180 degrees
- moved U$24 1.78 mm to (32.1, 11.4)
- moved U$2 1.78 mm to (27.9, 12.7)
- moved R2 1.27 mm to (15.2, 14.0)
- moved R5 0.64 mm to (24.8, 14.0)
- moved R6 0.63 mm to (19.1, 15.2)
- moved R1 0.63 mm to (22.9, 14.0)
- moved U$6 0.51 mm to (24.1, 10.2)
- moved U$1 0.51 mm to (28.2, 11.4)
Routing:
- net N$3: track 1.92 -> 3.95 mm
- net SDA: track 32.2 -> 33.3 mm
- net SCL: track 48.1 -> 47.2 mm
- net N$2: track 1.41 -> 2.04 mm
- net GND: track 2.00 -> 2.64 mm, vias 13 -> 10
- net ACK: track 4.57 -> 5.21 mm
Other:
- board text added: "v10"
- board text removed: "v01"
