File: Hardware/gator_UV.sch (EAGLE design)
At the start: 31 parts, among them J1 GATORGATOR_MINI, J2 GATORGATOR_MINI, J3 GATORGATOR_MINI, J4 GATORGATOR_MINI, J5 GATORGATOR_MINI, J6 GATORGATOR_MINI, J7 GATORGATOR_MINI, J8 GATORGATOR_MINI, Q1 2.5A/30V/105mΩ, U1 VEML6070"

Commit message: qc double check changes
Parts:
- U1: value VEML6070" -> VEML6070
Changed lines of the file:
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@@
 <part name="Q1" library="SparkFun-DiscreteSemi" deviceset="MOSFET_PCH" device="-DMG2307L" value="2.5A/30V/105mΩ"/>
 <part name="R4" library="SparkFun-Resistors" deviceset="10KOHM" device="-0603-1/10W-1%" value="10k"/>
-<part name="U1" library="SparkFun-Sensors" deviceset="VEML6070" device="&quot;"/>
+<part name="U1" library="SparkFun-Sensors" deviceset="VEML6070" device="&quot;" value="VEML6070"/>
 <part name="R5" library="SparkFun-Resistors" deviceset="10KOHM" device="-0603-1/10W-1%" value="10k"/>
 <part name="R6" library="SparkFun-Resistors" deviceset="300KOHM" device="-0603-1/10W-1%" value="300k"/>
